File: IPEPS_Elec/IPEPS_Elec.sch (KiCad schematic (older format))
At the start: 38 parts

Commit message: set the pull-down resistors values to 22k
Parts:
- R? (x4): value 10k -> 22k
Changed lines of the file:
@@
 P 3970 1675
 F 0 "R?" V 4040 1665 50  0000 C CNN
-F 1 "10k" V 3880 1675 50  0000 C CNN
+F 1 "22k" V 3880 1675 50  0000 C CNN
 F 2 "" H 3970 1675 50  0001 C CNN
 F 3 "~" H 3970 1675 50  0001 C CNN
@@
 P 3910 2230
 F 0 "R?" V 3980 2220 50  0000 C CNN
-F 1 "10k" V 3820 2230 50  0000 C CNN
+F 1 "22k" V 3820 2230 50  0000 C CNN
 F 2 "" H 3910 2230 50  0001 C CNN
 F 3 "~" H 3910 2230 50  0001 C CNN
@@
 P 3905 2765
 F 0 "R?" V 3975 2755 50  0000 C CNN
-F 1 "10k" V 3815 2765 50  0000 C CNN
+F 1 "22k" V 3815 2765 50  0000 C CNN
 F 2 "" H 3905 2765 50  0001 C CNN
 F 3 "~" H 3905 2765 50  0001 C CNN
@@
 P 6575 4225
 F 0 "R?" V 6645 4215 50  0000 C CNN
-F 1 "10k" V 6485 4225 50  0000 C CNN
+F 1 "22k" V 6485 4225 50  0000 C CNN
 F 2 "" H 6575 4225 50  0001 C CNN
 F 3 "~" H 6575 4225 50  0001 C CNN

Commit message: change label for C AND T
Connections:
- net C+T renamed C.T
Changed lines of the file:
@@
 	5085 2700 5085 2665
 Text GLabel 5765 2800 2    50   Input ~ 0
-C+T
+C.T
 Wire Wire Line
 	5730 2800 5765 2800
 Text GLabel 5075 4585 0    50   Input ~ 0
-C+T
+C.T
 Wire Wire Line
 	5075 4585 5135 4585

Commit message: fix pull-down values
Parts:
- R? (x4): value 22k -> 2.2k
Changed lines of the file:
@@
 P 3970 1675
 F 0 "R?" V 4040 1665 50  0000 C CNN
-F 1 "22k" V 3880 1675 50  0000 C CNN
+F 1 "2.2k" V 3880 1675 50  0000 C CNN
 F 2 "" H 3970 1675 50  0001 C CNN
 F 3 "~" H 3970 1675 50  0001 C CNN
@@
 P 3910 2230
 F 0 "R?" V 3980 2220 50  0000 C CNN
-F 1 "22k" V 3820 2230 50  0000 C CNN
+F 1 "2.2k" V 3820 2230 50  0000 C CNN
 F 2 "" H 3910 2230 50  0001 C CNN
 F 3 "~" H 3910 2230 50  0001 C CNN
@@
 P 3905 2765
 F 0 "R?" V 3975 2755 50  0000 C CNN
-F 1 "22k" V 3815 2765 50  0000 C CNN
+F 1 "2.2k" V 3815 2765 50  0000 C CNN
 F 2 "" H 3905 2765 50  0001 C CNN
 F 3 "~" H 3905 2765 50  0001 C CNN
@@
 P 6575 4225
 F 0 "R?" V 6645 4215 50  0000 C CNN
-F 1 "22k" V 6485 4225 50  0000 C CNN
+F 1 "2.2k" V 6485 4225 50  0000 C CNN
 F 2 "" H 6575 4225 50  0001 C CNN
 F 3 "~" H 6575 4225 50  0001 C CNN
